File: hardware/kicad_project/NN-antenna-manager.kicad_pcb (KiCad board)
At the start: 4 copper layers, 100.2 x 62.9 mm, 71 parts, among them IC1 PE42482A-X, J1 USB_C_Receptacle_USB2.0_16P, J10 Conn_Coaxial, J11 I2C Screen, J12 Serial, J2 Conn_Coaxial, J3 Conn_Coaxial, J4 Conn_Coaxial, J5 Conn_Coaxial, J6 Conn_Coaxial, J7 Conn_Coaxial, J8 Conn_Coaxial, J9 Conn_Coaxial, SW1 SW_Push, SW2 SW_Push, SW3 Button_up, SW4 Button_down, U1 USBLC6-2SC6, U2 AP2112K-3.3, U3 ESP32-C3-WROOM-02

Commit message: small fixes
Parts:
- moved SW3 13.6 mm to (123.4, 98.0)
- moved SW4 13.6 mm to (136.7, 98.0)
Routing:
- net Net-(R14-Pad2): track 10.5 -> 21.4 mm
- net Net-(R16-Pad2): track 10.5 -> 9.44 mm
Changed lines of the file:
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@@
 	(footprint "Button_Switch_SMD:SW_SPST_B3U-1000P"
 		(layer "F.Cu")
-		(at 136.66 84.406 180)
+		(at 136.66 97.9678 180)
 		(descr "Ultra-small-sized Tactile Switch with High Contact Reliability, Top-actuated Model, without Ground Terminal, without Boss")
 		(tags "Tactile Switch")
@@
 		(tags "capacitor handsolder")
 		(property "Reference" "C29"
-			(at 0 1.462 180)
+			(at 3.3328 -0.2652 180)
 			(layer "F.SilkS")
 			(effects
@@
 	(footprint "Button_Switch_SMD:SW_SPST_B3U-1000P"
 		(layer "F.Cu")
-		(at 123.4266 84.406 180)
+		(at 123.444 97.9678 180)
 		(descr "Ultra-small-sized Tactile Switch with High Contact Reliability, Top-actuated Model, without Ground Terminal, without Boss")
 		(tags "Tactile Switch")
@@
 	)
 	(segment
-		(start 134.8976 84.406)
-		(end 133.8072 85.4964)
-		(width 0.2032)
+		(start 134.96 97.9678)
+		(end 134.1374 97.9678)
+		(width 0.2)
 		(layer "F.Cu")
 		(net "Net-(R16-Pad2)")
@@
 	)
 	(segment
-		(start 134.96 84.406)
-		(end 134.8976 84.406)
-		(width 0.2032)
+		(start 131.8768 95.7072)
+		(end 131.9822 95.6018)
+		(width 0.2)
+		(layer "F.Cu")
+		(net "Net-(R16-Pad2)")
+	)
+	(segment
+		(start 131.9822 95.6018)
+		(end 131.9822 93.599)
+		(width 0.2)
 		(layer "F.Cu")
 		(net "Net-(R16-Pad2)")
@@
 	)
 	(segment
-		(start 131.9822 93.2142)
-		(end 131.9822 93.599)
-		(width 0.2032)
+		(start 134.1374 97.9678)
+		(end 131.8768 95.7072)
+		(width 0.2)
 		(layer "F.Cu")
 		(net "Net-(R16-Pad2)")
 	)
 	(segment
-		(start 133.8072 85.4964)
-		(end 133.8072 91.089)
+		(start 131.9822 93.2142)
+		(end 131.9822 93.599)
 		(width 0.2032)
 		(layer "F.Cu")
@@
 	)
 	(segment
+		(start 117.3226 89.4334)
+		(end 117.7544 89.0016)
+		(width 0.2)
+		(layer "F.Cu")
+		(net "Net-(R14-Pad2)")
+	)
+	(segment
+		(start 115.7224 94.7674)
+		(end 115.7224 91.6432)
+		(width 0.2)
+		(layer "F.Cu")
+		(net "Net-(R14-Pad2)")
+	)
+	(segment
 		(start 118.3424 93.1126)
 		(end 118.3424 93.5228)
@@
 	)
 	(segment
+		(start 119.634 89.027)
+		(end 120.2182 89.6112)
+		(width 0.2)
+		(layer "F.Cu")
+		(net "Net-(R14-Pad2)")
+	)
+	(segment
 		(start 120.1674 91.2876)
 		(end 118.3424 93.1126)
@@
 	)
 	(segment
-		(start 121.7266 84.406)
-		(end 120.3452 85.7874)
-		(width 0.2032)
+		(start 117.3226 90.043)
+		(end 117.3226 89.4334)
+		(width 0.2)
+		(layer "F.Cu")
+		(net "Net-(R14-Pad2)")
+	)
+	(segment
+		(start 120.1674 89.662)
+		(end 120.1674 91.0128)
+		(width 0.2)
 		(layer "F.Cu")
 		(net "Net-(R14-Pad2)")
@@
 	)
 	(segment
-		(start 120.3452 85.7874)
-		(end 120.3452 86.36)
-		(width 0.2032)
+		(start 121.744 97.9678)
+		(end 118.9228 97.9678)
+		(width 0.2)
 		(layer "F.Cu")
 		(net "Net-(R14-Pad2)")
 	)
 	(segment
-		(start 120.3452 86.36)
-		(end 120.1674 86.5378)
-		(width 0.2032)
+		(start 117.9576 89.0016)
+		(end 117.983 89.027)
+		(width 0.2)
 		(layer "F.Cu")
 		(net "Net-(R14-Pad2)")
 	)
 	(segment
-		(start 120.1674 86.5378)
-		(end 120.1674 91.0128)
-		(width 0.2032)
+		(start 117.7544 89.0016)
+		(end 117.9576 89.0016)
+		(width 0.2)
+		(layer "F.Cu")
+		(net "Net-(R14-Pad2)")
+	)
+	(segment
+		(start 115.7224 91.6432)
+		(end 117.3226 90.043)
+		(width 0.2)
+		(layer "F.Cu")
+		(net "Net-(R14-Pad2)")
+	)
+	(segment
+		(start 120.2182 89.6112)
+		(end 120.1674 89.662)
+		(width 0.2)
+		(layer "F.Cu")
+		(net "Net-(R14-Pad2)")
+	)
+	(segment
+		(start 117.983 89.027)
+		(end 119.634 89.027)
+		(width 0.2)
+		(layer "F.Cu")
+		(net "Net-(R14-Pad2)")
+	)
+	(segment
+		(start 118.9228 97.9678)
+		(end 115.7224 94.7674)
+		(width 0.2)
 		(layer "F.Cu")
 		(net "Net-(R14-Pad2)")
